File: apps/home_lab_manager/board/motherboard.brd (EAGLE design)
At the start: 100 x 80 mm, 18 parts, among them X1 22-23-2021

Commit message: Adding mq-2 gaz sensor (wip)
Parts:
- added C1: 100n, rcl:C0805
- added D2, D3: 1N4148, diode:DO-214AC
- added JP1: FAN1, pinhead:1X03
- added JP3: FAN1, pinhead:1X01
- added JP4: FAN2, pinhead:1X03
- added JP7: FAN2, pinhead:1X01
- added JP8: UI, pinhead:1X10
- added R1, R10, R13, R14, R6: 100k, rcl:R0805
- added R11, R2: 10k, rcl:R0805
- added R12, R5: 1k, rcl:R0805
- added R15: 20k, rcl:R0805
- added U$2: MQ_2, bzd:MQ_2
- added U$5, U$6: MGSF1N03L, bzd:SOT23_3_PIN
- JP6: value 5V -> 7V
Connections:
- new net 3.3V: JP8.1, JP8.9, U$1.PIN_0
- new net EINK_BUSY: JP8.8, U$1.PIN_12
- new net EINK_DC: JP8.6, U$1.PIN_9
- new net EINK_RST: JP8.7, U$1.PIN_11
- new net FAN1_SENSE: R1.1, R2.2, U$1.PIN_19
- new net FAN2_SENSE: R10.1, R11.2, U$1.PIN_18
- new net FAN_SWITCH: JP3.1, JP7.1, R12.1, R13.2, R5.1, R6.2, U$1.PIN_17
- new net GND_FAN1: D2.A, JP1.1, U$5.P$3
- new net GND_FAN2: D3.A, JP4.1, U$6.P$3
- new net I2C_SCL: U$1.PIN_13
- new net I2C_SDA: U$1.PIN_10
- new net N$1: JP1.3, R1.2
- new net N$2: R5.2, U$5.P$1
- new net N$3: JP4.3, R10.2
- new net N$4: R12.2, U$6.P$1
- new net N$5: U$2.A1, U$2.A2, U$2.H1
- new net N$6: C1.1, R15.2, U$2.B1, U$2.B2
- new net SPI_CLK: JP8.4, U$1.PIN_8
- new net SPI_CS0: JP8.5, U$1.PIN_7
- new net SPI_MOSI: JP8.3, U$1.PIN_14
- new net SWITCH: JP8.10, R14.2, U$1.PIN_5
- net GND: now also C1.2, JP8.2, R11.1, R13.1, R14.1, R15.1, R2.1, R6.1, U$2.H2, U$5.P$2, U$6.P$2
- net VIN_REG: now also D2.C, D3.C, JP1.2, JP4.2
Routing:
- net FAN_SWITCH: track 0.00 -> 17.9 mm
- net GND: track 45.2 -> 52.1 mm
- net GND_FAN2: track 0.00 -> 3.29 mm
- net GND_FAN1: track 0.00 -> 3.29 mm
- net N$4: track 0.00 -> 2.75 mm
- net N$2: track 0.00 -> 2.75 mm
Other:
- outline, holes or cut-outs redrawn
