File: apps/homelab_manager/board/motherboard.sch (EAGLE design)
At the start: 39 parts, among them X1 22-23-2021

Commit message: Adding components
Parts:
- removed JP8: UI, pinhead:PINHD-1X10
- added C3: 100n, rcl:C-EUC0805
- added C5: 10u, rcl:C-EUC0805
- added C6: 100u, rcl:C-EUC0805
- added JP10: LED, pinhead:PINHD-1X1
- added JP11: 5V, pinhead:PINHD-1X1
- added JP9: (no value), pinhead:PINHD-1X11
- added R16: 330, rcl:R-EU_R0805
- added R17: 5k, rcl:R-EU_R0805
- added R18: 1k, rcl:R-EU_R0805
- added R19: 100k, rcl:R-EU_R0805
- added U$8: MGSF1N03L, bzd:MGSF1N03L
- added U$9: LD1117, bzd:LD1117
- R15: value 20k -> 5k
Connections:
- removed net N$6: C1.1, R15.2, U$2.B1, U$2.B2
- new net 5V: C3.1, C6.1, JP11.1, U$2.A1, U$2.A2, U$2.H1, U$9.OUT
- new net GND_LED: JP9.11, R16.2
- new net LED: JP10.1, R18.1, R19.2
- new net N$14: R16.1, U$8.D
- new net N$7: JP9.9
- new net N$8: R18.2, U$8.G
- new net VOUT_GAZ: C1.1, R15.2, R17.1, U$1.23_GPIO25
- net 3.3V: now also JP9.1; no longer JP8.1, JP8.9
- net 7V: now also C5.1, U$9.IN
- net EINK_BUSY: now also JP9.8; no longer JP8.8
- net EINK_DC: now also JP9.6; no longer JP8.6
- net EINK_RST: now also JP9.7; no longer JP8.7
- net GND: now also C3.2, C5.2, C6.2, JP9.2, R19.1, U$8.S, U$9.GND; no longer JP8.2
- net N$5: now also R17.2, U$2.B1, U$2.B2; no longer U$2.A1, U$2.A2, U$2.H1
- net SPI_CLK: now also JP9.4; no longer JP8.4
- net SPI_CS0: now also JP9.5; no longer JP8.5
- net SPI_MOSI: now also JP9.3; no longer JP8.3
- net SWITCH: now also JP9.10; no longer JP8.10
Other:
- note added: "Comes with different part number for specific output voltage: - 1.2 V LD1117S12TR - 1.8 V LD1117S18TR - 2.5 V LD1117S25TR - 3.3 V LD1117S33TR - 5.0 V LD1117S50TR"
- moved on the sheet: C1, R14, R15

Commit message: Started main layout
Parts:
- added C7: 100n, rcl:C-EUC0805
- added D4: 1N4148, diode:DIODE-DO-214AC
- added JP12: HOMELAB, pinhead:PINHD-1X1
- added R21, R24: 100k, rcl:R-EU_R0805
- added R23: 1k, rcl:R-EU_R0805
- added RELAY: 22-23-2021, con-molex:22-23-2021
- added U$10: TMP101, bzd:TMP101
- added U$11: MGSF1N03L, bzd:MGSF1N03L
- renumbered X1 to DCIN
Connections:
- new net GND_RELAY: D4.A, RELAY-1.S, U$11.D
- new net HOMELAB_POWER: JP12.1, R23.1, R24.2, U$1.22_GPIO33
- new net N$13: R23.2, U$11.G
- new net TEMPERATURE_ALERT: R21.1, U$1.26_GPIO14, U$10.ALERT
- net 3.3V: now also C7.1, R21.2, U$10.V+
- net GND: now also C7.2, R24.1, U$10.ADD0, U$10.GND, U$11.S
- net I2C_SCL: now also U$10.SCL
- net I2C_SDA: now also U$10.SDA
- net LED: now also U$1.27_GPIO12
- net VIN_REG: now also D4.C, RELAY-2.S

Commit message: Updated bazelisk + bazel
Parts:
- removed DCIN: 22-23-2021, con-molex:22-23-2021
- added DC_12V: DC_POWER_2.1MM, bzd:DC_POWER_2.1MM
Connections:
- net 12V: now also DC_12V.V+; no longer DCIN-2.S
- net GND: now also DC_12V.V-; no longer DCIN-1.S
Changed lines of the file:
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@@
 <parts>
 <part name="U$1" library="bzd" deviceset="ESP32_DEVKIT_V1" device=""/>
-<part name="DCIN" library="con-molex" library_urn="urn:adsk.eagle:library:165" deviceset="22-23-2021" device="" package3d_urn="urn:adsk.eagle:package:8078633/1"/>
-<part name="GND6" library="supply1" library_urn="urn:adsk.eagle:library:371" deviceset="GND" device=""/>
 <part name="U$4" library="bzd" deviceset="TPS561201" device=""/>
 <part name="GND12" library="supply1" library_urn="urn:adsk.eagle:library:371" deviceset="GND" device=""/>
@@
 <part name="D4" library="diode" library_urn="urn:adsk.eagle:library:210" deviceset="DIODE-" device="DO-214AC" package3d_urn="urn:adsk.eagle:package:43416/2" value="1N4148"/>
 <part name="RELAY" library="con-molex" library_urn="urn:adsk.eagle:library:165" deviceset="22-23-2021" device="" package3d_urn="urn:adsk.eagle:package:8078633/1"/>
+<part name="DC_12V" library="bzd" deviceset="DC_POWER_2.1MM" device=""/>
+<part name="GND22" library="supply1" library_urn="urn:adsk.eagle:library:371" deviceset="GND" device=""/>
 </parts>
 <sheets>
@@
 <attribute name="NAME" x="55.88" y="35.56" size="1.778" layer="95"/>
 </instance>
-<instance part="DCIN" gate="-1" x="-101.6" y="83.82" smashed="yes" rot="R180">
-<attribute name="NAME" x="-104.14" y="84.582" size="1.524" layer="95" rot="R180"/>
-<attribute name="VALUE" x="-100.838" y="82.423" size="1.778" layer="96" rot="R180"/>
-</instance>
-<instance part="DCIN" gate="-2" x="-101.6" y="86.36" smashed="yes" rot="R180">
-<attribute name="NAME" x="-104.14" y="87.122" size="1.524" layer="95" rot="R180"/>
-</instance>
-<instance part="GND6" gate="1" x="-96.52" y="78.74" smashed="yes">
-<attribute name="VALUE" x="-99.06" y="76.2" size="1.778" layer="96"/>
-</instance>
 <instance part="U$4" gate="G$1" x="-66.04" y="25.4" smashed="yes">
 <attribute name="NAME" x="-71.12" y="38.1" size="1.27" layer="95"/>
@@
 <instance part="RELAY" gate="-2" x="152.4" y="71.12" smashed="yes" rot="R180">
 <attribute name="NAME" x="149.86" y="71.882" size="1.524" layer="95" rot="R180"/>
+</instance>
+<instance part="DC_12V" gate="G$1" x="-68.58" y="76.2" smashed="yes">
+<attribute name="NAME" x="-70.358" y="81.788" size="1.778" layer="95"/>
+</instance>
+<instance part="GND22" gate="1" x="-78.74" y="68.58" smashed="yes">
+<attribute name="VALUE" x="-81.28" y="66.04" size="1.778" layer="96"/>
 </instance>
 </instances>
@@
 <nets>
 <net name="GND" class="0">
-<segment>
-<pinref part="DCIN" gate="-1" pin="S"/>
-<pinref part="GND6" gate="1" pin="GND"/>
-<wire x1="-99.06" y1="83.82" x2="-96.52" y2="83.82" width="0.1524" layer="91"/>
-<wire x1="-96.52" y1="83.82" x2="-96.52" y2="81.28" width="0.1524" layer="91"/>
-</segment>
 <segment>
 <pinref part="U$4" gate="G$1" pin="GND"/>
@@
 <wire x1="167.64" y1="48.26" x2="170.18" y2="48.26" width="0.1524" layer="91"/>
 <junction x="170.18" y="48.26"/>
+</segment>
+<segment>
+<pinref part="DC_12V" gate="G$1" pin="V-"/>
+<wire x1="-76.2" y1="73.66" x2="-78.74" y2="73.66" width="0.1524" layer="91"/>
+<pinref part="GND22" gate="1" pin="GND"/>
+<wire x1="-78.74" y1="73.66" x2="-78.74" y2="71.12" width="0.1524" layer="91"/>
 </segment>
 </net>
@@
 <net name="12V" class="0">
 <segment>
-<pinref part="DCIN" gate="-2" pin="S"/>
-<wire x1="-99.06" y1="86.36" x2="-83.82" y2="86.36" width="0.1524" layer="91"/>
-<label x="-91.44" y="86.36" size="1.778" layer="95"/>
-</segment>
-<segment>
 <pinref part="U$3" gate="G$1" pin="VIN+"/>
 <pinref part="R3" gate="G$1" pin="1"/>
@@
 <label x="-91.44" y="-53.34" size="1.778" layer="95"/>
 </segment>
+<segment>
+<pinref part="DC_12V" gate="G$1" pin="V+"/>
+<wire x1="-76.2" y1="78.74" x2="-86.36" y2="78.74" width="0.1524" layer="91"/>
+<label x="-86.36" y="78.74" size="1.778" layer="95"/>
+</segment>
 </net>

Commit message: motherboard (wip)
Parts:
- added JP8: SWITCH_LED, pinhead:PINHD-1X3
- added RELAY1: 22-23-2021, con-molex:22-23-2021
- added U$12, U$13: SCREW_TERMINAL, bzd:SCREW_TERMINAL
- added U$7: RELAY_SONGLE, bzd:RELAY_SONGLE
- JP9: value (none) -> UI
Connections:
- removed net N$7: JP9.9
- new net N$15: RELAY1-1.S, U$7.COMMAND_V-
- new net N$16: U$12.2, U$13.1
- new net N$17: U$12.1, U$7.V-
- new net N$18: U$13.2, U$7.ACTIVE_V+
- new net N$6: RELAY1-2.S, U$7.COMMAND_V+
- net 3.3V: now also JP9.9
- net FAN2_SENSE: now also U$1.22_GPIO33; no longer U$1.19_GPIO34
- net HOMELAB_POWER: now also U$1.5_GPIO4; no longer U$1.22_GPIO33
- net LED: now also U$1.7_GPIO17; no longer U$1.27_GPIO12
- net VOUT_CURRENT: now also U$1.19_GPIO34; no longer U$1.5_GPIO4
Changed lines of the file:
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@@
 <part name="R19" library="rcl" library_urn="urn:adsk.eagle:library:334" deviceset="R-EU_" device="R0805" package3d_urn="urn:adsk.eagle:package:23553/2" value="100k"/>
 <part name="JP10" library="pinhead" library_urn="urn:adsk.eagle:library:325" deviceset="PINHD-1X1" device="" package3d_urn="urn:adsk.eagle:package:22485/2" value="LED"/>
-<part name="JP9" library="pinhead" library_urn="urn:adsk.eagle:library:325" deviceset="PINHD-1X11" device="" package3d_urn="urn:adsk.eagle:package:22410/2"/>
+<part name="JP9" library="pinhead" library_urn="urn:adsk.eagle:library:325" deviceset="PINHD-1X11" device="" package3d_urn="urn:adsk.eagle:package:22410/2" value="UI"/>
 <part name="R16" library="rcl" library_urn="urn:adsk.eagle:library:334" deviceset="R-EU_" device="R0805" package3d_urn="urn:adsk.eagle:package:23553/2" value="330"/>
 <part name="U$9" library="bzd" deviceset="LD1117" device=""/>
@@
 <part name="DC_12V" library="bzd" deviceset="DC_POWER_2.1MM" device=""/>
 <part name="GND22" library="supply1" library_urn="urn:adsk.eagle:library:371" deviceset="GND" device=""/>
+<part name="RELAY1" library="con-molex" library_urn="urn:adsk.eagle:library:165" deviceset="22-23-2021" device="" package3d_urn="urn:adsk.eagle:package:8078633/1"/>
+<part name="U$7" library="bzd" deviceset="RELAY_SONGLE" device=""/>
+<part name="U$12" library="bzd" deviceset="SCREW_TERMINAL" device=""/>
+<part name="U$13" library="bzd" deviceset="SCREW_TERMINAL" device=""/>
+<part name="JP8" library="pinhead" library_urn="urn:adsk.eagle:library:325" deviceset="PINHD-1X3" device="" package3d_urn="urn:adsk.eagle:package:22458/2" value="SWITCH_LED"/>
 </parts>
 <sheets>
@@
 <attribute name="VALUE" x="-81.28" y="66.04" size="1.778" layer="96"/>
 </instance>
+<instance part="RELAY1" gate="-1" x="195.58" y="68.58" smashed="yes" rot="R180">
+<attribute name="NAME" x="193.04" y="69.342" size="1.524" layer="95" rot="R180"/>
+<attribute name="VALUE" x="196.342" y="67.183" size="1.778" layer="96" rot="R180"/>
+</instance>
+<instance part="RELAY1" gate="-2" x="195.58" y="71.12" smashed="yes" rot="R180">
+<attribute name="NAME" x="193.04" y="71.882" size="1.524" layer="95" rot="R180"/>
+</instance>
+<instance part="U$7" gate="G$1" x="215.9" y="55.88" smashed="yes">
+<attribute name="NAME" x="219.964" y="71.882" size="1.778" layer="95"/>
+</instance>
+<instance part="U$12" gate="G$1" x="243.84" y="78.74" smashed="yes" rot="R90">
+<attribute name="NAME" x="238.252" y="79.502" size="1.778" layer="95" rot="R90"/>
+</instance>
+<instance part="U$13" gate="G$1" x="243.84" y="33.02" smashed="yes" rot="R270">
+<attribute name="NAME" x="249.428" y="32.258" size="1.778" layer="95" rot="R270"/>
+</instance>
+<instance part="JP8" gate="A" x="157.48" y="2.54" smashed="yes" rot="R180">
+<attribute name="NAME" x="163.83" y="-3.175" size="1.778" layer="95" rot="R180"/>
+<attribute name="VALUE" x="163.83" y="10.16" size="1.778" layer="96" rot="R180"/>
+</instance>
 </instances>
 <busses>
@@
 </segment>
 <segment>
-<pinref part="U$1" gate="G$1" pin="5_GPIO4"/>
-<wire x1="33.02" y1="66.04" x2="7.62" y2="66.04" width="0.1524" layer="91"/>
-<label x="7.62" y="66.04" size="1.778" layer="95"/>
+<pinref part="U$1" gate="G$1" pin="19_GPIO34"/>
+<wire x1="83.82" y1="48.26" x2="101.6" y2="48.26" width="0.1524" layer="91"/>
+<label x="93.98" y="48.26" size="1.778" layer="95"/>
 </segment>
 </net>
@@
 <net name="FAN2_SENSE" class="0">
 <segment>
-<pinref part="U$1" gate="G$1" pin="19_GPIO34"/>
-<wire x1="83.82" y1="48.26" x2="101.6" y2="48.26" width="0.1524" layer="91"/>
-<label x="93.98" y="48.26" size="1.778" layer="95"/>
-</segment>
-<segment>
 <pinref part="R10" gate="G$1" pin="1"/>
 <pinref part="R11" gate="G$1" pin="2"/>
@@
 <junction x="53.34" y="-45.72"/>
 <label x="55.88" y="-45.72" size="1.778" layer="95"/>
+</segment>
+<segment>
+<pinref part="U$1" gate="G$1" pin="22_GPIO33"/>
+<wire x1="83.82" y1="55.88" x2="101.6" y2="55.88" width="0.1524" layer="91"/>
+<label x="93.98" y="55.88" size="1.778" layer="95"/>
 </segment>
 </net>
@@
 <junction x="165.1" y="109.22"/>
 <label x="170.18" y="109.22" size="1.778" layer="95"/>
+</segment>
+<segment>
+<wire x1="-20.32" y1="114.3" x2="-40.64" y2="114.3" width="0.1524" layer="91"/>
+<label x="-40.64" y="114.3" size="1.778" layer="95"/>
+<pinref part="JP9" gate="A" pin="9"/>
 </segment>
 </net>
@@
 </segment>
 <segment>
-<pinref part="U$1" gate="G$1" pin="27_GPIO12"/>
-<wire x1="83.82" y1="68.58" x2="96.52" y2="68.58" width="0.1524" layer="91"/>
-<label x="91.44" y="68.58" size="1.778" layer="95"/>
-</segment>
-</net>
-<net name="N$7" class="0">
-<segment>
-<wire x1="-20.32" y1="114.3" x2="-40.64" y2="114.3" width="0.1524" layer="91"/>
-<label x="-40.64" y="114.3" size="1.778" layer="95"/>
-<pinref part="JP9" gate="A" pin="9"/>
+<pinref part="U$1" gate="G$1" pin="7_GPIO17"/>
+<wire x1="33.02" y1="60.96" x2="7.62" y2="60.96" width="0.1524" layer="91"/>
+<label x="7.62" y="60.96" size="1.778" layer="95"/>
 </segment>
 </net>
@@
 </segment>
 <segment>
-<pinref part="U$1" gate="G$1" pin="22_GPIO33"/>
-<wire x1="83.82" y1="55.88" x2="101.6" y2="55.88" width="0.1524" layer="91"/>
-<label x="93.98" y="55.88" size="1.778" layer="95"/>
-</segment>
-</net>
+<pinref part="U$1" gate="G$1" pin="5_GPIO4"/>
+<wire x1="33.02" y1="66.04" x2="7.62" y2="66.04" width="0.1524" layer="91"/>
+<label x="7.62" y="66.04" size="1.778" layer="95"/>
+</segment>
+</net>
+<net name="N$6" class="0">
+<segment>
+<pinref part="RELAY1" gate="-2" pin="S"/>
+<wire x1="198.12" y1="71.12" x2="198.12" y2="76.2" width="0.1524" layer="91"/>
+<pinref part="U$7" gate="G$1" pin="COMMAND_V+"/>
+<wire x1="198.12" y1="76.2" x2="215.9" y2="76.2" width="0.1524" layer="91"/>
+<wire x1="215.9" y1="76.2" x2="215.9" y2="73.66" width="0.1524" layer="91"/>
+</segment>
+</net>
+<net name="N$15" class="0">
+<segment>
+<pinref part="RELAY1" gate="-1" pin="S"/>
+<wire x1="198.12" y1="68.58" x2="198.12" y2="40.64" width="0.1524" layer="91"/>
+<wire x1="198.12" y1="40.64" x2="215.9" y2="40.64" width="0.1524" layer="91"/>
+<pinref part="U$7" gate="G$1" pin="COMMAND_V-"/>
+<wire x1="215.9" y1="40.64" x2="215.9" y2="43.18" width="0.1524" layer="91"/>
+</segment>
+</net>
+<net name="N$16" class="0">
+<segment>
+<pinref part="U$12" gate="G$1" pin="2"/>
+<pinref part="U$13" gate="G$1" pin="1"/>
+<wire x1="246.38" y1="73.66" x2="246.38" y2="38.1" width="0.1524" layer="91"/>
+</segment>
+</net>
+<net name="N$17" class="0">
+<segment>
+<pinref part="U$12" gate="G$1" pin="1"/>
+<wire x1="241.3" y1="73.66" x2="241.3" y2="58.42" width="0.1524" layer="91"/>
+<pinref part="U$7" gate="G$1" pin="V-"/>
+<wire x1="241.3" y1="58.42" x2="228.6" y2="58.42" width="0.1524" layer="91"/>
+</segment>
+</net>
+<net name="N$18" class="0">
+<segment>
+<pinref part="U$7" gate="G$1" pin="ACTIVE_V+"/>
+<wire x1="228.6" y1="50.8" x2="241.3" y2="50.8" width="0.1524" layer="91"/>
+<pinref part="U$13" gate="G$1" pin="2"/>
+<wire x1="241.3" y1="50.8" x2="241.3" y2="38.1" width="0.1524" layer="91"/>
+</segment>
+</net>

Commit message: Completed layout rev 1
Parts:
- added LED: LED, pinhead:PINHD-1X2
- added U$14: MOMENTARY_SWITCH, bzd:MOMENTARY_SWITCH
- renumbered JP8 to SWITCH_LED
Connections:
- new net N$19: LED.2, SWITCH_LED.1
- new net N$20: SWITCH_LED.2, U$14.P$1
- new net N$7: LED.1, SWITCH_LED.3, U$14.P$2
Changed lines of the file:
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@@
 <part name="U$12" library="bzd" deviceset="SCREW_TERMINAL" device=""/>
 <part name="U$13" library="bzd" deviceset="SCREW_TERMINAL" device=""/>
-<part name="JP8" library="pinhead" library_urn="urn:adsk.eagle:library:325" deviceset="PINHD-1X3" device="" package3d_urn="urn:adsk.eagle:package:22458/2" value="SWITCH_LED"/>
+<part name="SWITCH_LED" library="pinhead" library_urn="urn:adsk.eagle:library:325" deviceset="PINHD-1X3" device="" package3d_urn="urn:adsk.eagle:package:22458/2" value="SWITCH_LED"/>
+<part name="LED" library="pinhead" library_urn="urn:adsk.eagle:library:325" deviceset="PINHD-1X2" device="" package3d_urn="urn:adsk.eagle:package:22435/2" value="LED"/>
+<part name="U$14" library="bzd" deviceset="MOMENTARY_SWITCH" device=""/>
 </parts>
 <sheets>
@@
 <attribute name="NAME" x="249.428" y="32.258" size="1.778" layer="95" rot="R270"/>
 </instance>
-<instance part="JP8" gate="A" x="157.48" y="2.54" smashed="yes" rot="R180">
+<instance part="SWITCH_LED" gate="A" x="157.48" y="2.54" smashed="yes" rot="R180">
 <attribute name="NAME" x="163.83" y="-3.175" size="1.778" layer="95" rot="R180"/>
 <attribute name="VALUE" x="163.83" y="10.16" size="1.778" layer="96" rot="R180"/>
+</instance>
+<instance part="LED" gate="G$1" x="193.04" y="2.54" smashed="yes">
+<attribute name="NAME" x="186.69" y="8.255" size="1.778" layer="95"/>
+<attribute name="VALUE" x="186.69" y="-2.54" size="1.778" layer="96"/>
+</instance>
+<instance part="U$14" gate="G$1" x="170.18" y="2.54" smashed="yes">
+<attribute name="NAME" x="167.894" y="0.254" size="1.778" layer="95"/>
 </instance>
 </instances>
@@
 </segment>
 </net>
+<net name="N$7" class="0">
+<segment>
+<pinref part="SWITCH_LED" gate="A" pin="3"/>
+<pinref part="LED" gate="G$1" pin="1"/>
+<wire x1="160.02" y1="5.08" x2="175.26" y2="5.08" width="0.1524" layer="91"/>
+<pinref part="U$14" gate="G$1" pin="P$2"/>
+<wire x1="175.26" y1="5.08" x2="190.5" y2="5.08" width="0.1524" layer="91"/>
+<wire x1="175.26" y1="2.54" x2="175.26" y2="5.08" width="0.1524" layer="91"/>
+<junction x="175.26" y="5.08"/>
+</segment>
+</net>
+<net name="N$19" class="0">
+<segment>
+<pinref part="SWITCH_LED" gate="A" pin="1"/>
+<wire x1="160.02" y1="0" x2="177.8" y2="0" width="0.1524" layer="91"/>
+<wire x1="177.8" y1="0" x2="177.8" y2="2.54" width="0.1524" layer="91"/>
+<pinref part="LED" gate="G$1" pin="2"/>
+<wire x1="177.8" y1="2.54" x2="190.5" y2="2.54" width="0.1524" layer="91"/>
+</segment>
+</net>
+<net name="N$20" class="0">
+<segment>
+<pinref part="U$14" gate="G$1" pin="P$1"/>
+<pinref part="SWITCH_LED" gate="A" pin="2"/>
+<wire x1="165.1" y1="2.54" x2="160.02" y2="2.54" width="0.1524" layer="91"/>
+</segment>
+</net>
