File: kicad/jardinier2000/jardinier2000.kicad_pcb (KiCad board)
At the start: 2 copper layers, 53 parts, among them J1 5V, J10 I2C, J11 I2C, J2 VIN Reg, J3 5V, J4 5V, J5 5V, J6 5_30V, J7 I2C, J8 5V, J9 I2C, Q1 AO3400A, Q2 AO3400A, Q3 AO3400A, Q4 AO3400A, Q5 AO3400A, Q6 AO3400A, U1 ESP32_DevKit_V1_DOIT, U2 NCP1117-3.3_SOT223, U3 TPS62933P

Commit message: Working on pcb
Parts:
- added J12: Barrel_Jack_Switch, Connector_BarrelJack:BarrelJack_Horizontal, F.Cu at (97.0, 121.0)

Commit message: Routing of triggers
Parts:
- moved J8 107.1 mm to (80.0, 44.7), turned to 180 degrees
- moved L2 105.2 mm to (84.0, 44.7), turned to 180 degrees
- moved C11 102.9 mm to (80.0, 48.7), turned to -90 degrees
- moved C12 101.4 mm to (82.5, 48.7), turned to -90 degrees
- moved R7 98.4 mm to (86.0, 52.2)
- moved R8 98.0 mm to (87.5, 48.7), turned to 90 degrees
- moved U3 97.5 mm to (91.5, 49.2), turned to 90 degrees
- moved J2 97.4 mm to (86.0, 60.7), turned to 180 degrees
- moved R6 96.7 mm to (87.0, 56.2), turned to 180 degrees
- moved C1 94.8 mm to (85.0, 48.7), turned to -90 degrees
- moved C9 93.1 mm to (89.5, 45.2), turned to 180 degrees
- moved C10 90.2 mm to (93.5, 45.2)
- moved C8 88.6 mm to (91.5, 52.7)
- moved R2 88.2 mm to (118.8, 53.0), turned to 90 degrees
- moved D6 88.0 mm to (125.8, 53.0), turned to -90 degrees
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Routing:
- net /5V: track 0.00 -> 103.2 mm
- net GND: track 0.00 -> 62.9 mm, vias 0 -> 1
- net /VDD_5_30V: track 0.00 -> 21.2 mm
- net Net-(U3-SW): track 0.00 -> 15.3 mm
- net /MOSFET 3A/V-: track 0.00 -> 14.1 mm
- net /MOSFET 3A1/V-: track 0.00 -> 13.2 mm
- net /MOSFET 3A3/V-: track 0.00 -> 13.1 mm
- net /MOSFET 3A2/V-: track 0.00 -> 13.1 mm
- net Net-(U3-EN): track 0.00 -> 9.61 mm
- net Net-(U3-FB): track 0.00 -> 6.26 mm
- net /MOSFET 3A/Trigger: track 0.00 -> 4.04 mm
- net Net-(Q2-G): track 0.00 -> 3.87 mm
- net Net-(Q1-G): track 0.00 -> 3.87 mm
- net Net-(U3-BST): track 0.00 -> 3.59 mm
- net /MOSFET 3A3/Trigger: track 0.00 -> 3.54 mm
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
Commit message: Finished routing v1.0
Parts:
- added R18: 10K, Resistor_SMD:R_0805_2012Metric_Pad1.20x1.40mm_HandSolder, F.Cu at (154.0, 81.5)
- added R19: 10K, Resistor_SMD:R_0805_2012Metric_Pad1.20x1.40mm_HandSolder, F.Cu at (154.0, 68.5)
- added SW1: SW_Push, Button_Switch_THT:SW_PUSH_6mm, F.Cu at (159.2, 81.8)
- added SW2: SW_Push, Button_Switch_THT:SW_PUSH_6mm, F.Cu at (159.2, 68.2)
- J10, J11, J7, J9: footprint TerminalBlock_Phoenix:TerminalBlock_Phoenix_MKDS-1,5-4-5.08_1x04_P5.08mm_Horizontal -> Connector_JST:JST_XH_B4B-XH-AM_1x04_P2.50mm_Vertical
- J3: value 5V -> 5_30V
- J6: value 5_30V -> 5V
- moved J6 110.4 mm to (165.0, 44.0), turned to 180 degrees
- moved D1 103.5 mm to (83.5, 73.5)
- moved Q6 97.4 mm to (88.5, 75.2), turned to 180 degrees
- moved D5 93.1 mm to (164.9, 52.8), turned to -90 degrees
- moved R13 89.9 mm to (157.4, 52.8), turned to 90 degrees
- moved R17 89.6 mm to (91.0, 80.2), turned to 180 degrees
- moved R16 88.4 mm to (92.5, 75.7), turned to -90 degrees
- moved R12 88.4 mm to (160.9, 56.3), turned to 180 degrees
- moved Q5 87.6 mm to (160.9, 52.8), turned to 90 degrees
- moved C3 87.5 mm to (83.5, 76.5)
- moved C4 78.9 mm to (90.5, 85.2), turned to 90 degrees
- moved U2 77.8 mm to (85.0, 83.2), turned to -90 degrees
- moved R15 68.3 mm to (102.5, 97.5)
- moved R14 67.3 mm to (102.5, 100.0)
- moved J7 59.7 mm to (109.0, 105.0), turned to 90 degrees
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Connections:
- C3 pad 1: /MOSFET 3A5/V+ -> /5V
- D1 pad 1: /MOSFET 3A5/V+ -> /5V
- D2 pad 1: /5V -> /VDD_5_30V
- D5 pad 1: /VDD_5_30V -> /5V
- J3 pad 1: /5V -> /VDD_5_30V
- J6 pad 1: /VDD_5_30V -> /5V
- U1 pad 16: unconnected-(U1-3V3-Pad16) -> /ESP32_3V3
- U1 pad 18: unconnected-(U1-IO15-Pad18) -> /Trigger_3V3
- U1 pad 9: /Trigger_3V3 -> unconnected-(U1-IO26-Pad9)
- U2 pad 3: /MOSFET 3A5/V+ -> /5V
Routing:
- net GND: track 62.9 -> 349.3 mm, vias 1 -> 9
- net /5V: track 103.2 -> 221.5 mm
- net /3V3: track 0.00 -> 72.5 mm
- net /ESP32_3V3: track 0.00 -> 64.8 mm, vias 0 -> 2
- net /SDA: track 0.00 -> 48.9 mm
- net /SCL: track 0.00 -> 44.9 mm
- net /VDD_5_30V: track 21.2 -> 65.2 mm
- net /MOSFET 3A4/Trigger: track 0.00 -> 35.3 mm
- net /Trigger_3V3: track 0.00 -> 29.3 mm
- net /MOSFET 3A3/Trigger: track 3.54 -> 31.0 mm
- net /MOSFET 3A1/Trigger: track 3.54 -> 20.1 mm
- net /MOSFET 3A2/Trigger: track 3.54 -> 19.8 mm
- net /MOSFET 3A4/V-: track 0.00 -> 13.1 mm
- net /MOSFET 3A5/V-: track 0.00 -> 11.8 mm
- net Net-(R19-Pad2): track 0.00 -> 10.9 mm
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- added copper zone on B.Cu, net GND
Other:
- board outline added: 103.5 x 72.5 mm
- board text added: "3V3"
- board text added: "5-30V"
- board text added: "5V"
- board text added: "GND"
- board text added: "Jardinier2000 v1.0 bzd"
- board text added: "POWER"
- board text added: "POWER 6-30V"
- board text added: "SCL"
- board text added: "SDA"

Commit message: Updating schematics for v2
Parts:
- removed C10: 100n & 3A, Capacitor_SMD:C_0805_2012Metric_Pad1.18x1.45mm_HandSolder
- removed C11: 10u, Capacitor_SMD:C_0805_2012Metric_Pad1.18x1.45mm_HandSolder
- removed C12, C8: 0.1u, Capacitor_SMD:C_0805_2012Metric_Pad1.18x1.45mm_HandSolder
- removed C9: 33n, Capacitor_SMD:C_0805_2012Metric_Pad1.18x1.45mm_HandSolder
- removed D5: D_Schottky, Diode_SMD:D_0805_2012Metric_Pad1.15x1.40mm_HandSolder
- removed J10: I2C, Connector_JST:JST_XH_B4B-XH-AM_1x04_P2.50mm_Vertical
- removed J8: 5V, Connector_PinHeader_1.00mm:PinHeader_1x01_P1.00mm_Vertical
- removed L2: 6.8uH & 3A, Inductor_SMD:L_1008_2520Metric_Pad1.43x2.20mm_HandSolder
- removed Q5, Q6: AO3400A, Package_TO_SOT_SMD:SOT-23
- removed R10, R12, R14, R15: 10K, Resistor_SMD:R_0805_2012Metric_Pad1.20x1.40mm_HandSolder
- removed R11, R13: 100, Resistor_SMD:R_0805_2012Metric_Pad1.20x1.40mm_HandSolder
- removed SW1, SW2: SW_Push, Button_Switch_THT:SW_PUSH_6mm
- removed U3: TPS62933P, Package_TO_SOT_SMD:SOT-583-8
- added C13: 0.1u, Capacitor_SMD:C_0805_2012Metric_Pad1.18x1.45mm_HandSolder, F.Cu at (125.9, 128.6)
- added C14: 0.1u, Capacitor_SMD:C_0805_2012Metric_Pad1.18x1.45mm_HandSolder, F.Cu at (78.0, 76.1)
- added C15: 0.1u, Capacitor_SMD:C_0805_2012Metric_Pad1.18x1.45mm_HandSolder, F.Cu at (78.0, 79.1)
- added C16: 0.1u, Capacitor_SMD:C_0805_2012Metric_Pad1.18x1.45mm_HandSolder, F.Cu at (78.0, 82.1)
- added C17: 2.2u, Capacitor_SMD:C_0805_2012Metric_Pad1.18x1.45mm_HandSolder, F.Cu at (65.1, 134.1)
- added C18: 0.1u, Capacitor_SMD:C_0805_2012Metric_Pad1.18x1.45mm_HandSolder, F.Cu at (65.1, 137.1)
- added C19: 10u, Capacitor_SMD:C_0805_2012Metric_Pad1.18x1.45mm_HandSolder, F.Cu at (65.1, 140.1)
- added C2: 0.1u, Capacitor_SMD:C_0805_2012Metric_Pad1.18x1.45mm_HandSolder, F.Cu at (125.9, 116.5)
- added C20: 10u, Capacitor_SMD:C_0805_2012Metric_Pad1.18x1.45mm_HandSolder, F.Cu at (65.1, 143.1)
- added C5: 0.1u, Capacitor_SMD:C_0805_2012Metric_Pad1.18x1.45mm_HandSolder, F.Cu at (125.9, 125.6)
- added C6: 0.1u, Capacitor_SMD:C_0805_2012Metric_Pad1.18x1.45mm_HandSolder, F.Cu at (78.0, 73.1)
- added D7: D_Schottky, Diode_SMD:D_0805_2012Metric_Pad1.15x1.40mm_HandSolder, F.Cu at (84.0, 124.0)
- added D8: LED, LED_SMD:LED_0805_2012Metric_Pad1.15x1.40mm_HandSolder, F.Cu at (65.1, 150.1)
- added J14: USB_C_Receptacle_USB2.0_16P, Connector_USB:USB_C_Receptacle_G-Switch_GT-USB-7010ASV, F.Cu at (136.7, 122.9)
- added JP1: SolderJumper_3_Open, Jumper:SolderJumper-3_P1.3mm_Open_Pad1.0x1.5mm_NumberLabels, F.Cu at (115.5, 137.5)
- added JP2: SolderJumper_3_Open, Jumper:SolderJumper-3_P1.3mm_Open_Pad1.0x1.5mm_NumberLabels, F.Cu at (115.5, 141.1)
- added JP3: SolderJumper_3_Open, Jumper:SolderJumper-3_P1.3mm_Open_Pad1.0x1.5mm_NumberLabels, F.Cu at (115.5, 144.6)
- added JP4: SolderJumper_3_Open, Jumper:SolderJumper-3_P1.3mm_Open_Pad1.0x1.5mm_NumberLabels, F.Cu at (115.5, 148.2)
- added L1: 3.3uH & 3A, Inductor_SMD:L_Cenker_CKCS6028, F.Cu at (75.7, 136.4)
- added R20: 10K, Resistor_SMD:R_0805_2012Metric_Pad1.20x1.40mm_HandSolder, F.Cu at (78.0, 88.0)
- added R21: 10K, Resistor_SMD:R_0805_2012Metric_Pad1.20x1.40mm_HandSolder, F.Cu at (78.0, 91.0)
- added R22: 5.1K, Resistor_SMD:R_0805_2012Metric_Pad1.20x1.40mm_HandSolder, F.Cu at (133.2, 129.1)
- added R23: 5.1K, Resistor_SMD:R_0805_2012Metric_Pad1.20x1.40mm_HandSolder, F.Cu at (133.2, 132.1)
- added SW3: RESET, bzd:push_button_6x3, F.Cu at (102.0, 87.0)
- added SW4: SW_Push, Button_Switch_THT:SW_PUSH_6mm, F.Cu at (67.1, 73.6)
- added SW5: SW_Push, Button_Switch_THT:SW_PUSH_6mm, F.Cu at (67.1, 82.2)
- added SW6: SW_Push, Button_Switch_THT:SW_PUSH_6mm, F.Cu at (67.1, 90.7)
- added TP1: 3V3, TestPoint:TestPoint_Pad_2.0x2.0mm, F.Cu at (66.0, 109.8)
- added TP2: VIN, TestPoint:TestPoint_Pad_2.0x2.0mm, F.Cu at (66.0, 113.9)
- added TP3: VBUS, TestPoint:TestPoint_Pad_2.0x2.0mm, F.Cu at (66.0, 118.0)
- added TP4: VIN_LDO_3V3, TestPoint:TestPoint_Pad_2.0x2.0mm, F.Cu at (66.0, 122.0)
- added TP5: VIN_STEP_DOWN, TestPoint:TestPoint_Pad_2.0x2.0mm, F.Cu at (69.6, 134.6)
- added TP6: VOUT_STEP_DOWN, TestPoint:TestPoint_Pad_2.0x2.0mm, F.Cu at (69.6, 138.6)
- added U4: ESP32-S3-WROOM-1, RF_Module:ESP32-S3-WROOM-1, F.Cu at (118.3, 88.4)
- C1: value 22u -> 0.1u
- C7: value 10u -> 0.1u
- J1, J4: value 5V -> ~
- J2: value VIN Reg -> ~; footprint Connector_PinHeader_1.00mm:PinHeader_1x01_P1.00mm_Vertical -> TerminalBlock_Phoenix:TerminalBlock_Phoenix_MKDS-1,5-2-5.08_1x02_P5.08mm_Horizontal
- J3: value 5_30V -> ~
- J5, J6: value 5V -> ADC; footprint TerminalBlock_Phoenix:TerminalBlock_Phoenix_MKDS-1,5-2-5.08_1x02_P5.08mm_Horizontal -> Connector_JST:JST_XH_B3B-XH-AM_1x03_P2.50mm_Vertical
- J9: value I2C -> Screw_Terminal_01x06; footprint Connector_JST:JST_XH_B4B-XH-AM_1x04_P2.50mm_Vertical -> Connector_JST:JST_XH_B6B-XH-AM_1x06_P2.50mm_Vertical
- R17: value 100 -> 10K
- R18: value 10K -> 100k
- R19: value 10K -> 13.7k
- R6: value 1M -> 1k
- R7: value 10.2K -> 10K
- R8: value 53.6K -> 100
- U1: value ESP32_DevKit_V1_DOIT -> LMR51430YDDCR; footprint bzd:esp32_devkit_v1_doit -> Package_TO_SOT_SMD:SOT-23-6
- moved J6 118.5 mm to (73.1, 118.7), turned to 0 degrees
- moved R19 113.7 mm to (69.9, 145.1)
- moved R8 111.1 mm to (115.1, 156.4), turned to 0 degrees
- moved R7 105.3 mm to (115.1, 153.4)
- moved R18 103.7 mm to (69.9, 142.1)
- moved J5 102.3 mm to (73.1, 110.9), turned to 0 degrees
- moved U1 94.7 mm to (74.9, 143.1), turned to 0 degrees
- moved J2 88.9 mm to (121.9, 142.0), turned to 0 degrees
- moved R4 88.0 mm to (147.2, 126.3), turned to 0 degrees
- moved D2 88.0 mm to (152.0, 128.0), turned to 0 degrees
- moved Q2 87.1 mm to (152.0, 124.3), turned to 0 degrees
- moved R3 80.7 mm to (147.2, 123.3), turned to 0 degrees
- moved J12 76.1 mm to (138.0, 107.8)
- moved J4 68.7 mm to (85.1, 90.1), turned to 0 degrees
- moved D4 65.6 mm to (152.0, 118.3), turned to 0 degrees
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Connections:
- net Net-(U3-FB) renamed /TRIG3
- C1 pad 1: /5V -> /ADC1_CH0
- C3 pad 1: /5V -> Net-(D1-K)
- C3 pad 2: /MOSFET 3A5/V- -> GND
- C4 pad 1: /3V3 -> 3V3
- C7 pad 1: /VDD_5_30V -> /ADC2_CH0
- D1 pad 1: /5V -> Net-(D1-K)
- D1 pad 2: /MOSFET 3A5/V- -> VCC_5V
- D2 pad 1: /VDD_5_30V -> /MOSFET 3A1/V+
- D3 pad 1: /5V -> /MOSFET 3A2/V+
- D4 pad 1: /5V -> /MOSFET 3A3/V+
- D6 pad 1: /5V -> /MOSFET 3A/V+
- J1 pad 1: /5V -> /MOSFET 3A/V+
- J11 pad 2: /3V3 -> 3V3
- J12 pad 1: /VDD_5_30V -> VIN
- J2 pad 1: /VDD_5_30V -> /MOSFET 3A3/V+
- J3 pad 1: /VDD_5_30V -> /MOSFET 3A1/V+
- J4 pad 1: /5V -> /MOSFET 3A2/V+
- J5 pad 1: /5V -> GND
- J5 pad 2: /MOSFET 3A3/V- -> 3V3
- J6 pad 1: /5V -> GND
- J6 pad 2: /MOSFET 3A4/V- -> 3V3
- J7 pad 2: /3V3 -> 3V3
- J9 pad 1: GND -> 3V3
- J9 pad 2: /3V3 -> /TCK
- J9 pad 3: /SDA -> /TDO
- J9 pad 4: /SCL -> /TDI
- R1 pad 2: /MOSFET 3A/Trigger -> /TRIG0
- R16 pad 1: GND -> 3V3
- R16 pad 2: /Trigger_3V3 -> /RESET
- R17 pad 1: /Trigger_3V3 -> 3V3
- R17 pad 2: Net-(Q6-G) -> /SW0
- R18 pad 1: /ESP32_3V3 -> VCC_5V
- R18 pad 2: Net-(R18-Pad2) -> Net-(U1-FB)
- R19 pad 1: /ESP32_3V3 -> Net-(U1-FB)
- R19 pad 2: Net-(R19-Pad2) -> GND
- R2 pad 1: /MOSFET 3A/Trigger -> /TRIG0
- R3 pad 2: /MOSFET 3A1/Trigger -> /TRIG1
- R4 pad 1: /MOSFET 3A1/Trigger -> /TRIG1
- R5 pad 2: /MOSFET 3A2/Trigger -> /TRIG2
- R6 pad 1: /VDD_5_30V -> /LED0
- R8 pad 2: /5V -> Net-(Q4-G)
- R9 pad 1: /MOSFET 3A2/Trigger -> /TRIG2
- U1 pad 1: unconnected-(U1-EN-Pad1) -> GND
- U1 pad 2: unconnected-(U1-SENSOR_VP-Pad2) -> Net-(U1-SW)
- U1 pad 3: unconnected-(U1-SENSOR_VN-Pad3) -> VIN
- U1 pad 4: unconnected-(U1-IO34-Pad4) -> Net-(U1-FB)
- U1 pad 5: unconnected-(U1-IO35-Pad5) -> VIN
- U1 pad 6: /MOSFET 3A4/Trigger -> Net-(U1-CB)
- U2 pad 1: /MOSFET 3A5/V- -> GND
- U2 pad 2: /3V3 -> 3V3
- U2 pad 3: /5V -> Net-(D1-K)
Routing:
- net GND: track 349.3 -> 0.00 mm, vias 9 -> 0
- net /5V: track 221.5 -> 0.00 mm
- net /3V3: track 72.5 -> 0.00 mm
- net /VDD_5_30V: track 65.2 -> 0.00 mm
- net /ESP32_3V3: track 64.8 -> 0.00 mm, vias 2 -> 0
- net /SDA: track 48.9 -> 0.00 mm
- net /SCL: track 44.9 -> 0.00 mm
- net /MOSFET 3A4/Trigger: track 35.3 -> 0.00 mm
- net /MOSFET 3A3/Trigger: track 31.0 -> 0.00 mm
- net /Trigger_3V3: track 29.3 -> 0.00 mm
- net /MOSFET 3A1/Trigger: track 20.1 -> 0.00 mm
- net /MOSFET 3A2/Trigger: track 19.8 -> 0.00 mm
- net Net-(U3-SW): track 15.3 -> 0.00 mm
- net /MOSFET 3A1/V-: track 13.2 -> 0.00 mm
- net /MOSFET 3A3/V-: track 13.1 -> 0.00 mm
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- removed copper zone on B.Cu, net GND
Other:
- board outline removed
- board text removed: "3V3"
- board text removed: "5-30V"
- board text removed: "5V"
- board text removed: "GND"
- board text removed: "Jardinier2000 v1.0 bzd"
- board text removed: "POWER"
- board text removed: "POWER 6-30V"
- board text removed: "SCL"
- board text removed: "SDA"

Commit message: jardinier2000 v0.2
Parts:
- removed TP2: VIN, TestPoint:TestPoint_Pad_2.0x2.0mm
- added G***: LOGO, LOGO, F.Cu at (142.4, 55.5)
- J5: value ADC -> ADC1_CH0
- J6: value ADC -> ADC2_CH0
- J9: value Screw_Terminal_01x06 -> JTAG
- moved J11 89.4 mm to (156.0, 61.8), turned to -90 degrees
- moved J5 87.8 mm to (155.4, 80.3), turned to 90 degrees
- moved J6 86.7 mm to (155.4, 91.4), turned to 90 degrees
- moved D8 85.0 mm to (116.4, 82.2)
- moved SW4 79.7 mm to (144.6, 92.0), turned to 90 degrees
- moved R8 72.1 mm to (158.4, 98.7), turned to -90 degrees
- moved J9 71.9 mm to (139.0, 74.2), turned to 90 degrees
- moved R7 71.7 mm to (157.5, 95.6)
- moved R17 70.9 mm to (148.9, 82.7), turned to 180 degrees
- moved C1 70.1 mm to (135.0, 61.0), turned to 90 degrees
- moved C13 69.4 mm to (112.6, 60.4), turned to 90 degrees
- moved SW5 69.2 mm to (135.6, 92.0), turned to 90 degrees
- moved J7 67.6 mm to (148.6, 61.8), turned to -90 degrees
- moved C14 67.2 mm to (144.9, 82.7), turned to 180 degrees
- moved R18 66.4 mm to (109.6, 88.9)
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Connections:
- U4 pad 20: unconnected-(U4-IO12-Pad20) -> /TRIG0
- U4 pad 21: unconnected-(U4-IO13-Pad21) -> /TRIG1
- U4 pad 22: unconnected-(U4-IO14-Pad22) -> /TRIG2
- U4 pad 23: /SW2 -> /TRIG3
- U4 pad 25: unconnected-(U4-IO48-Pad25) -> /SW2
- U4 pad 4: /TRIG0 -> unconnected-(U4-IO4-Pad4)
- U4 pad 5: /TRIG1 -> unconnected-(U4-IO5-Pad5)
- U4 pad 6: /TRIG2 -> unconnected-(U4-IO6-Pad6)
- U4 pad 7: /TRIG3 -> unconnected-(U4-IO7-Pad7)
Routing:
- net GND: track 0.00 -> 369.9 mm, vias 0 -> 12
- net 3V3: track 0.00 -> 181.4 mm, vias 0 -> 5
- net VCC_5V: track 0.00 -> 98.3 mm, vias 0 -> 5
- net VIN: track 0.00 -> 68.4 mm, vias 0 -> 4
- net /TRIG3: track 0.00 -> 48.5 mm, vias 0 -> 2
- net /SDA: track 0.00 -> 46.8 mm, vias 0 -> 2
- net /SCL: track 0.00 -> 43.9 mm, vias 0 -> 2
- net /TRIG2: track 0.00 -> 41.7 mm
- net /ADC2_CH0: track 0.00 -> 40.0 mm, vias 0 -> 1
- net /ADC1_CH0: track 0.00 -> 32.0 mm, vias 0 -> 1
- net /TRIG1: track 0.00 -> 30.6 mm
- net /SW0: track 0.00 -> 27.9 mm
- net VBUS_5V: track 0.00 -> 24.3 mm, vias 0 -> 2
- net /SW1: track 0.00 -> 20.9 mm
- net /TRIG0: track 0.00 -> 20.7 mm
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- added copper zone on B.Cu, net GND
Other:
- board outline added: 64 x 62 mm
- board text added: "ADC1 CH0"
- board text added: "ADC2 CH0"
- board text added: "I2C"
- board text added: "JTAG"
- board text added: "LED0"
- board text added: "RESET"
- board text added: "SW0"
- board text added: "SW1"
- board text added: "SW2"
- board text added: "TRIG0(VIN|5V)"
- board text added: "TRIG1(VIN|5V)"
- board text added: "TRIG2(VIN|5V)"
- board text added: "TRIG3(VIN|5V)"
- board text added: "VIN (6-36V)"
- board text added: "jardinier2000"
- board text added: "v0.2"
