File: kicad/jardinier2000/jardinier2000.kicad_sch (KiCad schematic)
At the start: 1 part, among them U1 ESP32_DevKit_V1_DOIT

Commit message: Updating design
Parts:
- added J1, J3, J4, J5: 5V, TerminalBlock_Phoenix:TerminalBlock_Phoenix_MKDS-1,5-2-5.08_1x02_P5.08mm_Horizontal, symbol Connector:Screw_Terminal_01x02
- added J6: 5_30V, TerminalBlock_Phoenix:TerminalBlock_Phoenix_MKDS-1,5-2-5.08_1x02_P5.08mm_Horizontal, symbol Connector:Screw_Terminal_01x02
Connections:
- net MOSFET 3A3/Trigger: now reaches U1.10 (IO27)
- net MOSFET 3A2/Trigger: now reaches U1.11 (IO14)
- net MOSFET 3A/Trigger: now reaches U1.12 (IO12)
- net MOSFET 3A1/Trigger: now reaches U1.13 (IO13)
- net GND: now reaches U1.14 (GND)
- net GND: now also U1.17 (GND)
- net 5V: now reaches U1.15 (VIN)
- net 5V: now also J1.1 (Pin_1), J3.1 (Pin_1), J4.1 (Pin_1), J5.1 (Pin_1)
- net MOSFET 3A4/Trigger: now reaches U1.6 (IO32)
- new net MOSFET 3A/V-: J1.2 (Pin_2)
- new net MOSFET 3A1/V-: J3.2 (Pin_2)
- new net MOSFET 3A2/V-: J4.2 (Pin_2)
- new net MOSFET 3A3/V-: J5.2 (Pin_2)
- new net MOSFET 3A4/V-: J6.2 (Pin_2)
- new net VDD_5_30V: J6.1 (Pin_1)
Other:
- added sheet MOSFET 3A (mosfet_3a.kicad_sch)
- added sheet MOSFET 3A1 (mosfet_3a.kicad_sch)
- added sheet MOSFET 3A2 (mosfet_3a.kicad_sch)
- added sheet MOSFET 3A3 (mosfet_3a.kicad_sch)
- added sheet MOSFET 3A4 (mosfet_3a.kicad_sch)
- added sheet Step Down 5V (step_down_5v.kicad_sch)

Commit message: Adding I2C
Parts:
- added C3, C4: 10u, Capacitor_SMD:C_0805_2012Metric_Pad1.18x1.45mm_HandSolder, symbol Device:C
- added J10, J11, J7, J9: I2C, TerminalBlock_Phoenix:TerminalBlock_Phoenix_MKDS-1,5-4-5.08_1x04_P5.08mm_Horizontal, symbol Connector:Screw_Terminal_01x04
- added R14, R15: 10K, Resistor_SMD:R_0805_2012Metric_Pad1.20x1.40mm_HandSolder, symbol Device:R
- added U2: NCP1117-3.3_SOT223, Package_TO_SOT_SMD:SOT-223-3_TabPin2, symbol Regulator_Linear:NCP1117-3.3_SOT223
Connections:
- net GND: now also C4.2, J10.4 (Pin_4), J11.4 (Pin_4), J7.4 (Pin_4), J9.4 (Pin_4)
- net SDA: now reaches U1.26 (IO21)
- net SDA: now also J10.2 (Pin_2), J11.2 (Pin_2), J7.2 (Pin_2), J9.2 (Pin_2), R14.2
- net SCL: now reaches U1.29 (IO22)
- net SCL: now also J10.3 (Pin_3), J11.3 (Pin_3), J7.3 (Pin_3), J9.3 (Pin_3), R15.2
- net Trigger_3V3: now reaches U1.9 (IO26)
- new net 3V3: C4.1, J10.1 (Pin_1), J11.1 (Pin_1), J7.1 (Pin_1), J9.1 (Pin_1), R14.1, R15.1, U2.2 (VO)
- new net MOSFET 3A5/V+: C3.1, U2.3 (VI)
- new net MOSFET 3A5/V-: C3.2, U2.1 (GND)
Other:
- added sheet MOSFET 3A5 (mosfet_3a.kicad_sch)

Commit message: Update bazel version
Parts:
- added J12: Barrel_Jack_Switch, Connector_BarrelJack:BarrelJack_Horizontal, symbol Connector:Barrel_Jack_Switch
Connections:
- net 3V3: now also J10.2 (Pin_2), J11.2 (Pin_2), J7.2 (Pin_2), J9.2 (Pin_2); no longer J10.1 (Pin_1), J11.1 (Pin_1), J7.1 (Pin_1), J9.1 (Pin_1)
- net GND: now also J10.1 (Pin_1), J11.1 (Pin_1), J7.1 (Pin_1), J9.1 (Pin_1), J12.1; no longer J10.4 (Pin_4), J11.4 (Pin_4), J7.4 (Pin_4), J9.4 (Pin_4)
- net SCL: now also J10.4 (Pin_4), J11.4 (Pin_4), J7.4 (Pin_4), J9.4 (Pin_4); no longer J10.3 (Pin_3), J11.3 (Pin_3), J7.3 (Pin_3), J9.3 (Pin_3)
- net SDA: now also J10.3 (Pin_3), J11.3 (Pin_3), J7.3 (Pin_3), J9.3 (Pin_3); no longer J10.2 (Pin_2), J11.2 (Pin_2), J7.2 (Pin_2), J9.2 (Pin_2)
- net VDD_5_30V: now also J12.2

Commit message: Working on pcb
Connections:
- net GND: now also J12.2; no longer J12.1
- net VDD_5_30V: now also J12.1; no longer J12.2
Changed lines of the file:
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@@
-	(wire
-		(pts
-			(xy 53.34 29.21) (xy 53.34 24.13)
-		)
-		(stroke
-			(width 0)
-			(type default)
-		)
-	)
 	(wire
 		(pts
@@
 	(wire
 		(pts
-			(xy 53.34 24.13) (xy 55.88 24.13)
-		)
-		(stroke
-			(width 0)
-			(type default)
-		)
-	)
-	(wire
-		(pts
 			(xy 107.95 146.05) (xy 107.95 154.94)
 		)
@@
 	(wire
 		(pts
-			(xy 50.8 34.29) (xy 58.42 34.29)
-		)
-		(stroke
-			(width 0)
-			(type default)
-		)
-	)
-	(wire
-		(pts
 			(xy 170.18 92.71) (xy 170.18 96.52)
 		)
@@
 	(wire
 		(pts
+			(xy 53.34 34.29) (xy 53.34 36.83)
+		)
+		(stroke
+			(width 0)
+			(type default)
+		)
+	)
+	(wire
+		(pts
 			(xy 132.08 93.98) (xy 142.24 93.98)
 		)
@@
 	(wire
 		(pts
+			(xy 50.8 34.29) (xy 53.34 34.29)
+		)
+		(stroke
+			(width 0)
+			(type default)
+		)
+	)
+	(wire
+		(pts
 			(xy 170.18 90.17) (xy 170.18 86.36)
 		)
@@
 		(pts
 			(xy 170.18 106.68) (xy 173.99 106.68)
-		)
-		(stroke
-			(width 0)
-			(type default)
-		)
-	)
-	(wire
-		(pts
-			(xy 55.88 24.13) (xy 55.88 26.67)
 		)
 		(stroke
@@
 	)
 	(label "VDD_5_30V"
-		(at 58.42 34.29 0)
+		(at 53.34 29.21 0)
 		(fields_autoplaced yes)
 		(effects
@@
 	(symbol
 		(lib_id "power:GND")
-		(at 55.88 26.67 0)
+		(at 53.34 36.83 0)
 		(unit 1)
 		(exclude_from_sim no)
@@
 		(fields_autoplaced yes)
 		(property "Reference" "#PWR028"
-			(at 55.88 33.02 0)
+			(at 53.34 43.18 0)
 			(effects
 				(font
@@
 		)
 		(property "Value" "GND"
-			(at 55.88 31.75 0)
+			(at 53.34 41.91 0)
 			(effects
 				(font
@@
 		)
 		(property "Footprint" ""
-			(at 55.88 26.67 0)
+			(at 53.34 36.83 0)
 			(effects
 				(font
@@
 		)
 		(property "Datasheet" ""
-			(at 55.88 26.67 0)
+			(at 53.34 36.83 0)
 			(effects
 				(font
@@
 		)
 		(property "Description" "Power symbol creates a global label with name \"GND\" , ground"
-			(at 55.88 26.67 0)
+			(at 53.34 36.83 0)
 			(effects
 				(font

Commit message: Finished routing v1.0
Parts:
- added R18, R19: 10K, Resistor_SMD:R_0805_2012Metric_Pad1.20x1.40mm_HandSolder, symbol Device:R
- added SW1, SW2: SW_Push, Button_Switch_THT:SW_PUSH_6mm, symbol Switch:SW_Push
- J10, J11, J7, J9: footprint TerminalBlock_Phoenix:TerminalBlock_Phoenix_MKDS-1,5-4-5.08_1x04_P5.08mm_Horizontal -> Connector_JST:JST_XH_B4B-XH-AM_1x04_P2.50mm_Vertical
- J3: value 5V -> 5_30V
- J6: value 5_30V -> 5V
Connections:
- net MOSFET 3A5/V+ is gone; now on net 5V: C3.1, U2.3 (VI)
- net 5V: now also J6.1 (Pin_1); no longer J3.1 (Pin_1)
- net GND: now also SW1.2, SW2.2
- net Trigger_3V3: now also U1.18 (IO15); no longer U1.9 (IO26)
- net VDD_5_30V: now also J3.1 (Pin_1); no longer J6.1 (Pin_1)
- net ESP32_3V3: now reaches U1.16 (3V3)
- net ESP32_3V3: now also R18.1, R19.1
- new net: R19.2, SW2.1
- new net: R18.2, SW1.1
Other:
- moved on the sheet: R14, R15

Commit message: Updating schematics for v2
Parts:
- removed J10, J9: I2C, Connector_JST:JST_XH_B4B-XH-AM_1x04_P2.50mm_Vertical, symbol Connector:Screw_Terminal_01x04
- removed J5, J6: 5V, TerminalBlock_Phoenix:TerminalBlock_Phoenix_MKDS-1,5-2-5.08_1x02_P5.08mm_Horizontal, symbol Connector:Screw_Terminal_01x02
- removed R14, R15, R18, R19: 10K, Resistor_SMD:R_0805_2012Metric_Pad1.20x1.40mm_HandSolder, symbol Device:R
- removed SW1, SW2: SW_Push, Button_Switch_THT:SW_PUSH_6mm, symbol Switch:SW_Push
- removed U1: ESP32_DevKit_V1_DOIT, bzd:esp32_devkit_v1_doit, symbol bzd:ESP32_DevKit_V1_DOIT
- added C1, C13, C14, C15, C16, C2, C5, C6, C7: 0.1u, Capacitor_SMD:C_0805_2012Metric_Pad1.18x1.45mm_HandSolder, symbol Device:C
- added D1, D7: D_Schottky, Diode_SMD:D_0805_2012Metric_Pad1.15x1.40mm_HandSolder, symbol Device:D_Schottky
- added D8: LED, LED_SMD:LED_0805_2012Metric_Pad1.15x1.40mm_HandSolder, symbol Device:LED
- added J14: USB_C_Receptacle_USB2.0_16P, Connector_USB:USB_C_Receptacle_G-Switch_GT-USB-7010ASV, symbol Connector:USB_C_Receptacle_USB2.0_16P
- added J2: ~, TerminalBlock_Phoenix:TerminalBlock_Phoenix_MKDS-1,5-2-5.08_1x02_P5.08mm_Horizontal, symbol Connector:Screw_Terminal_01x02
- added J5, J6: ADC, Connector_JST:JST_XH_B3B-XH-AM_1x03_P2.50mm_Vertical, symbol Connector:Screw_Terminal_01x03
- added J9: Screw_Terminal_01x06, Connector_JST:JST_XH_B6B-XH-AM_1x06_P2.50mm_Vertical, symbol Connector:Screw_Terminal_01x06
- added JP1, JP2, JP3, JP4: SolderJumper_3_Open, Jumper:SolderJumper-3_P1.3mm_Open_Pad1.0x1.5mm_NumberLabels, symbol Jumper:SolderJumper_3_Open
- added R16, R17, R20, R21: 10K, Resistor_SMD:R_0805_2012Metric_Pad1.20x1.40mm_HandSolder, symbol Device:R
- added R22, R23: 5.1K, Resistor_SMD:R_0805_2012Metric_Pad1.20x1.40mm_HandSolder, symbol Device:R
- added R6: 1k, Resistor_SMD:R_0805_2012Metric_Pad1.20x1.40mm_HandSolder, symbol Device:R
- added SW3: RESET, bzd:push_button_6x3, symbol Switch:SW_Push
- added SW4, SW5, SW6: SW_Push, Button_Switch_THT:SW_PUSH_6mm, symbol Switch:SW_Push
- added TP1: 3V3, TestPoint:TestPoint_Pad_2.0x2.0mm, symbol Connector:TestPoint
- added TP2: VIN, TestPoint:TestPoint_Pad_2.0x2.0mm, symbol Connector:TestPoint
- added TP3: VBUS, TestPoint:TestPoint_Pad_2.0x2.0mm, symbol Connector:TestPoint
- added TP4: VIN_LDO_3V3, TestPoint:TestPoint_Pad_2.0x2.0mm, symbol Connector:TestPoint
- added U4: ESP32-S3-WROOM-1, RF_Module:ESP32-S3-WROOM-1, symbol RF_Module:ESP32-S3-WROOM-1
- J1, J4: value 5V -> ~
- J3: value 5_30V -> ~
Connections:
- net MOSFET 3A5/V- is gone; now on net GND: C3.2, U2.1 (GND)
- net 3V3: now also C13.1, C5.1, J5.2 (Pin_2), J6.2 (Pin_2), J9.1 (Pin_1), R16.1, R17.1, R20.1, R21.1, TP1.1, U4.2 (3V3)
- net GND: now also C1.2, C13.2, C14.2, C15.2, C16.2, C2.2, C5.2, C6.2, C7.2, D8.1 (K), J14.A1 (GND), J14.A12 (GND), J14.B1 (GND), J14.B12 (GND), J14.S1 (SHIELD), J5.1 (Pin_1), J6.1 (Pin_1), J9.6 (Pin_6), R22.2, R23.2, SW3.1, SW4.1, SW5.1, SW6.1, U4.1 (GND), U4.40 (GND), U4.41 (GND)
- net MOSFET 3A3/V-: now also J2.2 (Pin_2)
- net SCL: now also U4.18 (IO10)
- net SDA: now also U4.17 (IO9)
- net 5V: no longer names the net of C3.1, U2.3 (VI)
- net 5V: now also C2.1, D1.1 (K), D7.1 (K), TP4.1; no longer J1.1 (Pin_1), J4.1 (Pin_1)
- net VDD_5_30V renamed MOSFET 3A1/V+
- net MOSFET 3A1/V+: now also JP2.2 (C); no longer J12.1
- new net: J14.B5 (CC2), R22.1
- new net: J14.A5 (CC1), R23.1
- new net: D8.2 (A), R6.2
- new net ADC1_CH0: C1.1, J5.3 (Pin_3), U4.39 (IO1)
- new net ADC2_CH0: C7.1, J6.3 (Pin_3), U4.19 (IO11)
- new net LED0: R6.1, U4.15 (IO3)
- new net MOSFET 3A/V+: J1.1 (Pin_1), JP1.2 (C)
- new net MOSFET 3A2/V+: J4.1 (Pin_1), JP3.2 (C)
- new net MOSFET 3A3/V+: J2.1 (Pin_1), JP4.2 (C)
- new net RESET: C6.1, R16.2, SW3.2, U4.3 (EN)
- new net SW0: C14.1, R17.2, SW4.2, U4.27 (IO0)
- new net SW1: C15.1, R20.2, SW5.2, U4.26 (IO45)
- new net SW2: C16.1, R21.2, SW6.2, U4.23 (IO21)
- new net TCK: J9.2 (Pin_2), U4.32 (IO39)
- new net TDI: J9.4 (Pin_4), U4.34 (IO41)
- new net TDO: J9.3 (Pin_3), U4.33 (IO40)
- new net TMS: J9.5 (Pin_5), U4.35 (IO42)
- new net TRIG0: U4.4 (IO4)
- new net TRIG1: U4.5 (IO5)
- new net TRIG2: U4.6 (IO6)
- new net TRIG3: U4.7 (IO7)
- new net USB_N: J14.A7 (D-), J14.B7 (D-), U4.13 (IO19)
- new net USB_P: J14.A6 (D+), J14.B6 (D+), U4.14 (IO20)
- new net VBUS_5V: D7.2 (A), J14.A4 (VBUS), J14.A9 (VBUS), J14.B4 (VBUS), J14.B9 (VBUS), TP3.1
- new net VCC_5V: D1.2 (A), JP1.3 (B), JP2.3 (B), JP3.3 (B), JP4.3 (B)
- new net VIN: J12.1, JP1.1 (A), JP2.1 (A), JP3.1 (A), JP4.1 (A), TP2.1
- no-connect marks 0 -> 21
Other:
- removed sheet MOSFET 3A4
- removed sheet MOSFET 3A5
- sheet Step Down 5V ports: added VIN_6_36V, VOUT_5V; removed VDD_5V, VDD_5_30V
- moved on the sheet: C3, C4, J1, J11, J3, J4, J7, U2

Commit message: jardinier2000 v0.2
Parts:
- removed TP2: VIN, TestPoint:TestPoint_Pad_2.0x2.0mm, symbol Connector:TestPoint
- J5: value ADC -> ADC1_CH0
- J6: value ADC -> ADC2_CH0
- J9: value Screw_Terminal_01x06 -> JTAG
Connections:
- net SW2: now also U4.25 (IO48); no longer U4.23 (IO21)
- net TRIG0: now also U4.20 (IO12); no longer U4.4 (IO4)
- net TRIG1: now also U4.21 (IO13); no longer U4.5 (IO5)
- net TRIG2: now also U4.22 (IO14); no longer U4.6 (IO6)
- net TRIG3: now also U4.23 (IO21); no longer U4.7 (IO7)
Other:
- note added: "ESP32-S3-WROOM-1: https://www.espressif.com/sites/default/files/documentation/esp32-s3-wroom-1_wroom-1u_datasheet_en.pdf"
Changed lines of the file:
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@@
 	)
 	(junction
-		(at 53.34 29.21)
-		(diameter 0)
-		(color 0 0 0 0)
-	)
-	(junction
 		(at 156.21 29.21)
 		(diameter 0)
@@
 	)
 	(no_connect
-		(at 99.06 107.95)
-	)
-	(no_connect
-		(at 99.06 105.41)
-	)
-	(no_connect
 		(at 99.06 80.01)
 	)
@@
 	)
 	(no_connect
+		(at 99.06 90.17)
+	)
+	(no_connect
+		(at 99.06 87.63)
+	)
+	(no_connect
+		(at 99.06 85.09)
+	)
+	(no_connect
 		(at 50.8 31.75)
 	)
@@
 	)
 	(no_connect
-		(at 99.06 110.49)
-	)
-	(no_connect
 		(at 99.06 113.03)
 	)
@@
 	)
 	(no_connect
-		(at 129.54 115.57)
+		(at 99.06 115.57)
 	)
 	(no_connect
-		(at 99.06 115.57)
+		(at 99.06 92.71)
 	)
 	(wire
@@
 	(wire
 		(pts
-			(xy 129.54 85.09) (xy 134.62 85.09)
-		)
-		(stroke
-			(width 0)
-			(type default)
-		)
-	)
-	(wire
-		(pts
 			(xy 83.82 168.91) (xy 81.28 168.91)
 		)
@@
 	(wire
 		(pts
-			(xy 85.09 87.63) (xy 99.06 87.63)
-		)
-		(stroke
-			(width 0)
-			(type default)
-		)
-	)
-	(wire
-		(pts
 			(xy 162.56 116.84) (xy 170.18 116.84)
 		)
@@
 	(wire
 		(pts
+			(xy 88.9 105.41) (xy 99.06 105.41)
+		)
+		(stroke
+			(width 0)
+			(type default)
+		)
+	)
+	(wire
+		(pts
 			(xy 129.54 82.55) (xy 134.62 82.55)
 		)
@@
 	(wire
 		(pts
-			(xy 46.99 156.21) (xy 49.53 156.21)
+			(xy 129.54 115.57) (xy 133.35 115.57)
 		)
 		(stroke
@@
 	(wire
 		(pts
-			(xy 85.09 85.09) (xy 99.06 85.09)
+			(xy 46.99 156.21) (xy 49.53 156.21)
 		)
 		(stroke
@@
 	(wire
 		(pts
+			(xy 88.9 107.95) (xy 99.06 107.95)
+		)
+		(stroke
+			(width 0)
+			(type default)
+		)
+	)
+	(wire
+		(pts
 			(xy 66.04 71.12) (xy 66.04 74.93)
 		)
@@
 	(wire
 		(pts
-			(xy 85.09 92.71) (xy 99.06 92.71)
-		)
-		(stroke
-			(width 0)
-			(type default)
-		)
-	)
-	(wire
-		(pts
 			(xy 38.1 132.08) (xy 36.83 132.08)
 		)
@@
 	(wire
 		(pts
+			(xy 88.9 110.49) (xy 99.06 110.49)
+		)
+		(stroke
+			(width 0)
+			(type default)
+		)
+	)
+	(wire
+		(pts
 			(xy 43.18 167.64) (xy 43.18 170.18)
 		)
@@
 	(wire
 		(pts
-			(xy 73.66 24.13) (xy 73.66 29.21)
+			(xy 129.54 85.09) (xy 134.62 85.09)
 		)
 		(stroke
@@
 	(wire
 		(pts
-			(xy 85.09 90.17) (xy 99.06 90.17)
+			(xy 73.66 24.13) (xy 73.66 29.21)
 		)
 		(stroke
@@
 	(wire
 		(pts
-			(xy 53.34 29.21) (xy 57.15 29.21)
-		)
-		(stroke
-			(width 0)
-			(type default)
-		)
-	)
-	(wire
-		(pts
 			(xy 58.42 181.61) (xy 63.5 181.61)
 		)
@@
 		)
 	)
+	(text "ESP32-S3-WROOM-1: https://www.espressif.com/sites/default/files/documentation/esp32-s3-wroom-1_wroom-1u_datasheet_en.pdf"
+		(exclude_from_sim no)
+		(at 216.408 152.908 0)
+		(effects
+			(font
+				(size 1.27 1.27)
+			)
+		)
+	)
 	(label "SCL"
 		(at 58.42 184.15 0)
@@
 		)
 	)
-	(label "SW2"
-		(at 134.62 85.09 0)
-		(fields_autoplaced yes)
-		(effects
-			(font
-				(size 1.27 1.27)
-			)
-			(justify left bottom)
-		)
-	)
 	(label "USB_N"
 		(at 134.62 80.01 0)
@@
 		)
 	)
-	(label "TRIG3"
-		(at 85.09 92.71 0)
-		(fields_autoplaced yes)
-		(effects
-			(font
-				(size 1.27 1.27)
-			)
-			(justify left bottom)
-		)
-	)
 	(label "ADC2_CH0"
 		(at 88.9 102.87 0)
@@
 		)
 	)
-	(label "SCL"
-		(at 92.71 100.33 0)
+	(label "TRIG1"
+		(at 88.9 107.95 0)
 		(fields_autoplaced yes)
 		(effects
@@
 		)
 	)
-	(label "TRIG2"
-		(at 85.09 90.17 0)
+	(label "SCL"
+		(at 92.71 100.33 0)
 		(fields_autoplaced yes)
 		(effects
@@
 		)
 	)
-	(label "SW0"
-		(at 85.09 74.93 0)
+	(label "TRIG0"
+		(at 88.9 105.41 0)
 		(fields_autoplaced yes)
 		(effects
@@
 		)
 	)
-	(label "SW1"
-		(at 134.62 107.95 0)
+	(label "SW2"
+		(at 133.35 115.57 0)
 		(fields_autoplaced yes)
 		(effects
@@
 		)
 	)
-	(label "USB_P"
-		(at 67.31 95.25 0)
+	(label "TRIG2"
+		(at 88.9 110.49 0)
 		(fields_autoplaced yes)
 		(effects
@@
 		)
 	)
-	(label "TRIG1"
-		(at 85.09 87.63 0)
+	(label "SW0"
+		(at 85.09 74.93 0)
+		(fields_autoplaced yes)
+		(effects
+			(font
+				(size 1.27 1.27)
+			)
+			(justify left bottom)
+		)
+	)
+	(label "SW1"
+		(at 134.62 107.95 0)
+		(fields_autoplaced yes)
+		(effects
+			(font
+				(size 1.27 1.27)
+			)
+			(justify left bottom)
+		)
+	)
+	(label "USB_P"
+		(at 67.31 95.25 0)
 		(fields_autoplaced yes)
 		(effects
@@
 		)
 	)
-	(label "TRIG0"
-		(at 85.09 85.09 0)
+	(label "SCL"
+		(at 40.64 184.15 0)
 		(fields_autoplaced yes)
 		(effects
@@
 		)
 	)
-	(label "SCL"
-		(at 40.64 184.15 0)
+	(label "TRIG3"
+		(at 134.62 85.09 0)
 		(fields_autoplaced yes)
 		(effects
@@
 			)
 		)
-		(property "Value" "ADC"
+		(property "Value" "ADC1_CH0"
 			(at 111.76 181.6099 0)
 			(effects
@@
 			)
 		)
-		(property "Value" "Screw_Terminal_01x06"
+		(property "Value" "JTAG"
 			(at 147.32 102.8699 0)
 			(effects
@@
 			)
 		)
-		(property "Value" "ADC"
+		(property "Value" "ADC2_CH0"
 			(at 91.44 181.6099 0)
 			(effects
@@
 					(unit 1)
 				)
-			)
-		)
-	)
-	(symbol
-		(lib_id "Connector:TestPoint")
-		(at 57.15 29.21 0)
-		(unit 1)
-		(exclude_from_sim no)
-		(in_bom yes)
-		(on_board yes)
-		(dnp no)
-		(fields_autoplaced yes)
-		(property "Reference" "TP2"
-			(at 59.69 24.6379 0)
-			(effects
-				(font
-					(size 1.27 1.27)
-				)
-				(justify left)
-			)
-		)
-		(property "Value" "VIN"
-			(at 59.69 27.1779 0)
-			(effects
-				(font
-					(size 1.27 1.27)
-				)
-				(justify left)
-			)
-		)
-		(property "Footprint" "TestPoint:TestPoint_Pad_2.0x2.0mm"
-			(at 62.23 29.21 0)
-			(effects
-				(font
-					(size 1.27 1.27)
-				)
-				(hide yes)
-			)
-		)
-		(property "Datasheet" "~"
-			(at 62.23 29.21 0)
-			(effects
-				(font
-					(size 1.27 1.27)
-				)
-				(hide yes)
-			)
-		)
-		(property "Description" "test point"
-			(at 57.15 29.21 0)
-			(effects
-				(font
-					(size 1.27 1.27)
-				)
-				(hide yes)
-			)
-		)
-		(pin "1"
-		)
-		(instances
-			(project "jardinier2000"
-				(path "/c98a1727-68a2-4147-9061-b7cb623ac6de"
-					(reference "TP2")
-					(unit 1)
-				)
