File: apps/jardinier2000/hardware/jardinier2000.kicad_sch (KiCad schematic)
At the start: 45 parts, among them J11 I2C, J12 Barrel_Jack_Switch, J14 USB_C_Receptacle_USB2.0_16P, J5 ADC1_CH0, J6 ADC2_CH0, J7 I2C, J9 JTAG, SW3 RESET, SW4 SW_Push, SW5 SW_Push, SW6 SW_Push, U2 NCP1117-3.3_SOT223, U4 ESP32-S3-WROOM-1

Commit message: Working on v0.3
Parts:
- J1, J2, J3, J4: value ~ -> (none)
Connections:
- net SW1: now also U4.24 (IO47); no longer U4.26 (IO45)
