File: apps/jardinier2000/hardware/step_down_5v.kicad_sch (KiCad schematic)
At the start: 10 parts, among them U1 LMR51430YDDCR

Commit message: Working on v0.3
Parts:
- added C21: 10u/50V, Capacitor_SMD:C_0805_2012Metric_Pad1.18x1.45mm_HandSolder, symbol Device:C
- added C22: 22u/50V/Electrolytic, Capacitor_THT:CP_Radial_D4.0mm_P1.50mm, symbol Device:C
- C17: value 2.2u -> 2.2u/50V
- C19, C20: value 10u -> 10u / 25V
- L1: value 3.3uH & 3A -> 4.7uH & 4A; footprint Inductor_SMD:L_Cenker_CKCS6028 -> Inductor_SMD:L_Cenker_CKCS8060
Connections:
- net GND: now also C21.2, C22.2
- net VIN_6_36V: now also C21.1, C22.1
